Commit message: Created a working version of the code to find the outer equation of the optimal reachable point basing on the mean of the reachability measure

File: src/reach_space_modeling/src/reach_space_modeling/generate_pointcloud/model/mobile_wx250s.urdf (robot description, URDF)
Before this commit: robot mobile_wx250s, 15 links, 14 joints
Links:
- link locobot/ar_tag_link: geometry collision mesh filename=/home/rosario/Desktop/base_pose_opt_ws/src/reach_space_mode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 scale=0.001 0.001 0.001; visual mesh filename=/home/rosario/Desktop/base_pose_opt_ws/src/reach_space_mode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 scale=0.001 0.001 0.001
- link locobot/arm_base_link: geometry collision mesh filename=/home/rosario/Desktop/base_pose_opt_ws/src/reach_space_mode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 scale=0.001 0.001 0.001; visual mesh filename=/home/rosario/Desktop/base_pose_opt_ws/src/reach_space_mode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 scale=0.001 0.001 0.001
- link locobot/gripper_bar_link: geometry collision mesh filename=/home/rosario/Desktop/base_pose_opt_ws/src/reach_space_mode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 scale=0.001 0.001 0.001; visual mesh filename=/home/rosario/Desktop/base_pose_opt_ws/src/reach_space_mode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 scale=0.001 0.001 0.001
- link locobot/gripper_link: geometry collision mesh filename=/home/rosario/Desktop/base_pose_opt_ws/src/reach_space_mode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 scale=0.001 0.001 0.001; visual mesh filename=/home/rosario/Desktop/base_pose_opt_ws/src/reach_space_mode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 scale=0.001 0.001 0.001
- link locobot/gripper_prop_link: geometry collision mesh filename=/home/rosario/Desktop/base_pose_opt_ws/src/reach_space_mode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 scale=0.001 0.001 0.001; visual mesh filename=/home/rosario/Desktop/base_pose_opt_ws/src/reach_space_mode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 scale=0.001 0.001 0.001
- link locobot/left_finger_link: geometry collision mesh filename=/home/rosario/Desktop/base_pose_opt_ws/src/reach_space_mode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 scale=0.001 0.001 0.001; visual mesh filename=/home/rosario/Desktop/base_pose_opt_ws/src/reach_space_mode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 scale=0.001 0.001 0.001
- link locobot/lower_forearm_link: geometry collision mesh filename=/home/rosario/Desktop/base_pose_opt_ws/src/reach_space_mode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 scale=0.001 0.001 0.001; visual mesh filename=/home/rosario/Desktop/base_pose_opt_ws/src/reach_space_mode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 scale=0.001 0.001 0.001
- link locobot/right_finger_link: geometry collision mesh filename=/home/rosario/Desktop/base_pose_opt_ws/src/reach_space_mode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 scale=0.001 0.001 0.001; visual mesh filename=/home/rosario/Desktop/base_pose_opt_ws/src/reach_space_mode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 scale=0.001 0.001 0.001
- link locobot/shoulder_link: geometry collision mesh filename=/home/rosario/Desktop/base_pose_opt_ws/src/reach_space_mode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 scale=0.001 0.001 0.001; visual mesh filename=/home/rosario/Desktop/base_pose_opt_ws/src/reach_space_mode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 scale=0.001 0.001 0.001
- link locobot/upper_arm_link: geometry collision mesh filename=/home/rosario/Desktop/base_pose_opt_ws/src/reach_space_mode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 scale=0.001 0.001 0.001; visual mesh filename=/home/rosario/Desktop/base_pose_opt_ws/src/reach_space_mode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 scale=0.001 0.001 0.001
- link locobot/upper_forearm_link: geometry collision mesh filename=/home/rosario/Desktop/base_pose_opt_ws/src/reach_space_mode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 scale=0.001 0.001 0.001; visual mesh filename=/home/rosario/Desktop/base_pose_opt_ws/src/reach_space_mode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 scale=0.001 0.001 0.001
- link locobot/wrist_link: geometry collision mesh filename=/home/rosario/Desktop/base_pose_opt_ws/src/reach_space_mode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 scale=0.001 0.001 0.001; visual mesh filename=/home/rosario/Desktop/base_pose_opt_ws/src/reach_space_mode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 scale=0.001 0.001 0.001

Commit message: minors

File: src/reach_space_modeling/src/reach_space_modeling/generate_pointcloud/model/mobile_wx250s.urdf (robot description, URDF)
Before this commit: robot mobile_wx250s, 15 links, 14 joints
Links:
- link locobot/ar_tag_link: geometry collision mesh filename=~/Desktop/base_pose_opt_ws/src/reach_space_modeling/src/rea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 scale=0.001 0.001 0.001; visual mesh filename=~/Desktop/base_pose_opt_ws/src/reach_space_modeling/src/rea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 scale=0.001 0.001 0.001
- link locobot/arm_base_link: geometry collision mesh filename=~/Desktop/base_pose_opt_ws/src/reach_space_modeling/src/rea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 scale=0.001 0.001 0.001; visual mesh filename=~/Desktop/base_pose_opt_ws/src/reach_space_modeling/src/rea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 scale=0.001 0.001 0.001
- link locobot/gripper_bar_link: geometry collision mesh filename=~/Desktop/base_pose_opt_ws/src/reach_space_modeling/src/rea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 scale=0.001 0.001 0.001; visual mesh filename=~/Desktop/base_pose_opt_ws/src/reach_space_modeling/src/rea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 scale=0.001 0.001 0.001
- link locobot/gripper_link: geometry collision mesh filename=~/Desktop/base_pose_opt_ws/src/reach_space_modeling/src/rea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 scale=0.001 0.001 0.001; visual mesh filename=~/Desktop/base_pose_opt_ws/src/reach_space_modeling/src/rea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 scale=0.001 0.001 0.001
- link locobot/gripper_prop_link: geometry collision mesh filename=~/Desktop/base_pose_opt_ws/src/reach_space_modeling/src/rea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 scale=0.001 0.001 0.001; visual mesh filename=~/Desktop/base_pose_opt_ws/src/reach_space_modeling/src/rea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 scale=0.001 0.001 0.001
- link locobot/left_finger_link: geometry collision mesh filename=~/Desktop/base_pose_opt_ws/src/reach_space_modeling/src/rea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 scale=0.001 0.001 0.001; visual mesh filename=~/Desktop/base_pose_opt_ws/src/reach_space_modeling/src/rea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 scale=0.001 0.001 0.001
- link locobot/lower_forearm_link: geometry collision mesh filename=~/Desktop/base_pose_opt_ws/src/reach_space_modeling/src/rea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 scale=0.001 0.001 0.001; visual mesh filename=~/Desktop/base_pose_opt_ws/src/reach_space_modeling/src/rea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 scale=0.001 0.001 0.001
- link locobot/right_finger_link: geometry collision mesh filename=~/Desktop/base_pose_opt_ws/src/reach_space_modeling/src/rea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 scale=0.001 0.001 0.001; visual mesh filename=~/Desktop/base_pose_opt_ws/src/reach_space_modeling/src/rea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 scale=0.001 0.001 0.001
- link locobot/shoulder_link: geometry collision mesh filename=~/Desktop/base_pose_opt_ws/src/reach_space_modeling/src/rea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 scale=0.001 0.001 0.001; visual mesh filename=~/Desktop/base_pose_opt_ws/src/reach_space_modeling/src/rea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 scale=0.001 0.001 0.001
- link locobot/upper_arm_link: geometry collision mesh filename=~/Desktop/base_pose_opt_ws/src/reach_space_modeling/src/rea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 scale=0.001 0.001 0.001; visual mesh filename=~/Desktop/base_pose_opt_ws/src/reach_space_modeling/src/rea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 scale=0.001 0.001 0.001
- link locobot/upper_forearm_link: geometry collision mesh filename=~/Desktop/base_pose_opt_ws/src/reach_space_modeling/src/rea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 scale=0.001 0.001 0.001; visual mesh filename=~/Desktop/base_pose_opt_ws/src/reach_space_modeling/src/rea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 scale=0.001 0.001 0.001
- link locobot/wrist_link: geometry collision mesh filename=~/Desktop/base_pose_opt_ws/src/reach_space_modeling/src/rea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 scale=0.001 0.001 0.001; visual mesh filename=~/Desktop/base_pose_opt_ws/src/reach_space_modeling/src/rea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 scale=0.001 0.001 0.001

Commit message: Fixed the problem with relative paths in mesh files of locobot URDF

File: src/reach_space_modeling/src/reach_space_modeling/generate_pointcloud/model/mobile_wx250s.urdf (robot description, URDF)
Before this commit: robot mobile_wx250s, 15 links, 14 joints
Links:
- link locobot/ar_tag_link: geometry collision mesh filename=meshes/mobile_wx250s_meshes/mobile_wx250s_11_ar_tag.stl scale=0.001 0.001 0.001; visual mesh filename=meshes/mobile_wx250s_meshes/mobile_wx250s_11_ar_tag.stl scale=0.001 0.001 0.001
- link locobot/arm_base_link: geometry collision mesh filename=meshes/mobile_wx250s_meshes/mobile_wx250s_1_base.stl scale=0.001 0.001 0.001; visual mesh filename=meshes/mobile_wx250s_meshes/mobile_wx250s_1_base.stl scale=0.001 0.001 0.001
- link locobot/gripper_bar_link: geometry collision mesh filename=meshes/mobile_wx250s_meshes/mobile_wx250s_9_gripper_bar.stl scale=0.001 0.001 0.001; visual mesh filename=meshes/mobile_wx250s_meshes/mobile_wx250s_9_gripper_bar.stl scale=0.001 0.001 0.001
- link locobot/gripper_link: geometry collision mesh filename=meshes/mobile_wx250s_meshes/mobile_wx250s_7_gripper.stl scale=0.001 0.001 0.001; visual mesh filename=meshes/mobile_wx250s_meshes/mobile_wx250s_7_gripper.stl scale=0.001 0.001 0.001
- link locobot/gripper_prop_link: geometry collision mesh filename=meshes/mobile_wx250s_meshes/mobile_wx250s_8_gripper_prop.stl scale=0.001 0.001 0.001; visual mesh filename=meshes/mobile_wx250s_meshes/mobile_wx250s_8_gripper_prop.stl scale=0.001 0.001 0.001
- link locobot/left_finger_link: geometry collision mesh filename=meshes/mobile_wx250s_meshes/mobile_wx250s_10_gripper_finger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 scale=0.001 0.001 0.001; visual mesh filename=meshes/mobile_wx250s_meshes/mobile_wx250s_10_gripper_finger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 scale=0.001 0.001 0.001
- link locobot/lower_forearm_link: geometry collision mesh filename=meshes/mobile_wx250s_meshes/mobile_wx250s_5_lower_forearm.s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 scale=0.001 0.001 0.001; visual mesh filename=meshes/mobile_wx250s_meshes/mobile_wx250s_5_lower_forearm.s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 scale=0.001 0.001 0.001
- link locobot/right_finger_link: geometry collision mesh filename=meshes/mobile_wx250s_meshes/mobile_wx250s_10_gripper_finger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 scale=0.001 0.001 0.001; visual mesh filename=meshes/mobile_wx250s_meshes/mobile_wx250s_10_gripper_finger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 scale=0.001 0.001 0.001
- link locobot/shoulder_link: geometry collision mesh filename=meshes/mobile_wx250s_meshes/mobile_wx250s_2_shoulder.stl scale=0.001 0.001 0.001; visual mesh filename=meshes/mobile_wx250s_meshes/mobile_wx250s_2_shoulder.stl scale=0.001 0.001 0.001
- link locobot/upper_arm_link: geometry collision mesh filename=meshes/mobile_wx250s_meshes/mobile_wx250s_3_upper_arm.stl scale=0.001 0.001 0.001; visual mesh filename=meshes/mobile_wx250s_meshes/mobile_wx250s_3_upper_arm.stl scale=0.001 0.001 0.001
- link locobot/upper_forearm_link: geometry collision mesh filename=meshes/mobile_wx250s_meshes/mobile_wx250s_4_upper_forearm.s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 scale=0.001 0.001 0.001; visual mesh filename=meshes/mobile_wx250s_meshes/mobile_wx250s_4_upper_forearm.s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 scale=0.001 0.001 0.001
- link locobot/wrist_link: geometry collision mesh filename=meshes/mobile_wx250s_meshes/mobile_wx250s_6_wrist.stl scale=0.001 0.001 0.001; visual mesh filename=meshes/mobile_wx250s_meshes/mobile_wx250s_6_wrist.stl scale=0.001 0.001 0.001
